File: pcb_design/bierdeckel.kicad_pcb (KiCad board)
At the start: 2 copper layers, 93 x 93 mm, 72 parts, among them IC1 HSFPAR004A, J1 Pogo, J2 Pogo, J6 USB-TYPE-C-020, Q1 BSS123, Q2 SP20P18T1, Q3 BSS123, SW1 PTS526 SK15 SMTR2 LFS, SW2 PTS526 SK15 SMTR2 LFS, SW3 PTS526 SK15 SMTR2 LFS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

Commit message: vendor more symbols
Parts:
- D2, D3, D4, D5: footprint LED_SMD:LED_WS2812B-2020_PLCC4_2.0x2.0mm -> bier:LED_WS2812B-2020_PLCC4_2.0x2.0mm
- IC1: footprint Samacsys:HSFPAR004A -> bier:HSFPAR004A
- SW1, SW2, SW3: footprint Button_Switch_SMD:SW_Push_1P1T_XKB_TS-1187A -> Button_Switch_SMD:SW_SPST_TL3342
- U6: footprint Snapeda:INA317IDGKR_SOP65P490X110-8N -> bier:INA317IDGKR_SOP65P490X110-8N
