File: pcb_design/bierdeckel.kicad_sch (KiCad schematic)
At the start: 33 parts, among them J1 Pogo, J2 Pogo, J6 USB-TYPE-C-020, Q1 BSS123, Q2 SP20P18T1, Q3 BSS123, SW1 PTS526 SK15 SMTR2 LFS, SW2 PTS526 SK15 SMTR2 LFS, SW3 PTS526 SK15 SMTR2 LFS, U1 ESP32-C3-WROOM-02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

Commit message: update PCB to Kicad 10
Parts:
- removed B1, B2, B3, B6: 0R, Resistor_SMD:R_1206_3216Metric, symbol Device:R
- added B1, B2, B3, B6: 0R, Resistor_SMD:R_1206_3216Metric, symbol Jumper:Jumper_2_Bridged
Connections:
- net GND: now also J6.SH (SHIELD), B1.1 (A), B1.2 (B), B2.1 (A), B2.2 (B), B3.1 (A), B3.2 (B), B6.1 (A), B6.2 (B); no longer J6.S1 (SHIELD)
Other:
- moved on the sheet: C32, C33, R1, R2, R3, R4

Commit message: vendor more symbols
Parts:
- SW1, SW2, SW3: footprint Button_Switch_SMD:SW_Push_1P1T_XKB_TS-1187A -> Button_Switch_SMD:SW_SPST_TL3342; symbol Switch:SW_Push -> bier:SW_Push_jumper
Changed lines of the file:
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@@
 	)
 	(symbol
-		(lib_id "Switch:SW_Push")
+		(lib_id "bier:SW_Push_jumper")
 		(at 101.6 44.45 0)
 		(unit 1)
@@
 			)
 		)
-		(property "Footprint" "Button_Switch_SMD:SW_Push_1P1T_XKB_TS-1187A"
+		(property "Footprint" "Button_Switch_SMD:SW_SPST_TL3342"
 			(at 101.6 39.37 0)
 			(hide yes)
@@
 		)
 		(property "Description" "Push button switch, generic, two pins"
-			(at 101.6 44.45 0)
+			(at 101.6 46.228 0)
 			(hide yes)
 			(show_name no)
@@
 		)
 		(property "part#" "PTS526 SK15 SMTR2 LFS"
-			(at 101.6 44.45 0)
+			(at 102.362 48.26 0)
 			(hide yes)
 			(show_name no)
@@
 		)
 		(property "mpn" "PTS526 SK15 SMTR2 LFS"
-			(at 101.6 44.45 0)
+			(at 101.854 51.308 0)
 			(hide yes)
 			(show_name no)
@@
 	)
 	(symbol
-		(lib_id "Switch:SW_Push")
+		(lib_id "bier:SW_Push_jumper")
 		(at 219.71 50.8 0)
 		(unit 1)
@@
 			)
 		)
-		(property "Footprint" "Button_Switch_SMD:SW_Push_1P1T_XKB_TS-1187A"
+		(property "Footprint" "Button_Switch_SMD:SW_SPST_TL3342"
 			(at 219.71 45.72 0)
 			(hide yes)
@@
 		)
 		(property "Description" "Push button switch, generic, two pins"
-			(at 219.71 50.8 0)
+			(at 219.71 52.578 0)
 			(hide yes)
 			(show_name no)
@@
 		)
 		(property "part#" "PTS526 SK15 SMTR2 LFS"
-			(at 219.71 50.8 0)
+			(at 220.472 54.61 0)
 			(hide yes)
 			(show_name no)
@@
 		)
 		(property "mpn" "PTS526 SK15 SMTR2 LFS"
-			(at 219.71 50.8 0)
+			(at 219.964 57.658 0)
 			(hide yes)
 			(show_name no)
@@
 	)
 	(symbol
-		(lib_id "Switch:SW_Push")
+		(lib_id "bier:SW_Push_jumper")
 		(at 200.66 46.99 90)
 		(unit 1)
@@
 			)
 		)
-		(property "Footprint" "Button_Switch_SMD:SW_Push_1P1T_XKB_TS-1187A"
+		(property "Footprint" "Button_Switch_SMD:SW_SPST_TL3342"
 			(at 195.58 46.99 0)
 			(hide yes)
@@
 		)
 		(property "Description" "Push button switch, generic, two pins"
-			(at 200.66 46.99 0)
+			(at 202.438 46.99 0)
 			(hide yes)
 			(show_name no)
@@
 		)
 		(property "part#" "PTS526 SK15 SMTR2 LFS"
-			(at 200.66 46.99 0)
+			(at 204.47 46.228 0)
 			(hide yes)
 			(show_name no)
@@
 		)
 		(property "mpn" "PTS526 SK15 SMTR2 LFS"
-			(at 200.66 46.99 0)
+			(at 207.518 46.736 0)
 			(hide yes)
 			(show_name no)
