File: pcb_design/pressure.kicad_sch (KiCad schematic)
At the start: 9 parts, among them IC1 HSFPAR004A, U6 INA317IDGKR

Commit message: vendor more symbols
Parts:
- IC1: symbol Samacsys:HSFPAR004A -> bier:HSFPAR004A
- U6: footprint Snapeda:INA317IDGKR_SOP65P490X110-8N -> bier:INA317IDGKR_SOP65P490X110-8N; symbol Snapeda:INA317IDGKR -> bier:INA317IDGKR
Changed lines of the file:
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@@
 	)
 	(symbol
-		(lib_id "Snapeda:INA317IDGKR")
+		(lib_id "bier:INA317IDGKR")
 		(at 133.35 59.69 0)
 		(unit 1)
@@
 			)
 		)
-		(property "Footprint" "Snapeda:INA317IDGKR_SOP65P490X110-8N"
+		(property "Footprint" "bier:INA317IDGKR_SOP65P490X110-8N"
 			(at 133.35 59.69 0)
 			(hide yes)
@@
 	)
 	(symbol
-		(lib_id "Samacsys:HSFPAR004A")
+		(lib_id "bier:HSFPAR004A")
 		(at 49.53 43.18 0)
 		(unit 1)
